Commit message: Update URDF files to match DC motor RS-555 specs (40-80 RPM, 2.5A rated current)
- Reduce wheel joint velocity from 10.0 to 1.4 rad/s (matching 40-80 RPM)
- Reduce wheel joint effort from 10.0 to 3.0 Nm (matching 2.5A current rating)
- Update Gazebo plugin limits for realistic motor performance
- Reduce arm servo joint velocities to 0.3-0.5 rad/s for realistic movement
- Adjust joint efforts to match servo capabilities

File: source/rpi/ros2-robosort/src/robosort_description/urdf/gazebo_control.xacro (robot description, xacro)
@@ -14,6 +14,6 @@
             <wheel_diameter>0.3048</wheel_diameter>        <!-- 12 inches (2 x wheel_radius) -->
             <!-- Limits -->
-            <max_wheel_torque>200</max_wheel_torque>
-            <max_wheel_acceleration>10.0</max_wheel_acceleration>
+            <max_wheel_torque>3.0</max_wheel_torque>
+            <max_wheel_acceleration>0.5</max_wheel_acceleration>
             <!-- Output -->
             <!-- Odometry frame and base frame -->

File: source/rpi/ros2-robosort/src/robosort_description/urdf/robosort.urdf.xacro (robot description, xacro)
@@ -129,6 +129,6 @@
       <origin xyz="-0.2524 ${reflect*wheel_separation/2} ${-body_height/2}" rpy="0 0 0"/>
       <axis xyz="0 1 0"/>
-      <limit effort="10.0" velocity="10.0"/>
-      <dynamics damping="0.1" friction="0.1"/>
+      <limit effort="3.0" velocity="1.4"/>
+      <dynamics damping="0.5" friction="0.3"/>
     </joint>
   </xacro:macro>
@@ -211,5 +211,5 @@
     <kd>100.0</kd>
     <minDepth>0.001</minDepth>
-    <maxVel>1.0</maxVel>
+    <maxVel>1.4</maxVel>
   </gazebo>
   <gazebo reference="right_wheel_link">
@@ -220,5 +220,5 @@
     <kd>100.0</kd>
     <minDepth>0.001</minDepth>
-    <maxVel>1.0</maxVel>
+    <maxVel>1.4</maxVel>
   </gazebo>
   <gazebo reference="front_left_caster_link">
@@ -249,6 +249,6 @@
       <wheel_diameter>${2*wheel_radius}</wheel_diameter>
       <!-- Limits -->
-      <max_wheel_torque>10.0</max_wheel_torque>
-      <max_wheel_acceleration>1.0</max_wheel_acceleration>
+      <max_wheel_torque>3.0</max_wheel_torque>
+      <max_wheel_acceleration>0.5</max_wheel_acceleration>
       <!-- Topic names -->
       <command_topic>cmd_vel</command_topic>

File: source/rpi/ros2-robosort/src/robosort_description/urdf/robosort_arm.urdf.xacro (robot description, xacro)
@@ -57,5 +57,5 @@
     <origin xyz="0 0 ${base_height}" rpy="0 0 0"/>
     <axis xyz="0 0 1"/>
-    <limit lower="${-PI}" upper="${PI}" effort="10.0" velocity="1.0"/>
+    <limit lower="${-PI}" upper="${PI}" effort="2.0" velocity="0.5"/>
   </joint>
   <!-- Shoulder Link (Servo 1) -->
@@ -85,5 +85,5 @@
     <origin xyz="0 0 ${shoulder_length}" rpy="0 0 0"/>
     <axis xyz="0 1 0"/>
-    <limit lower="${-PI/2}" upper="${PI/2}" effort="10.0" velocity="1.0"/>
+    <limit lower="${-PI/2}" upper="${PI/2}" effort="2.0" velocity="0.5"/>
   </joint>
   <!-- Elbow Link (Servo 2) -->
@@ -113,5 +113,5 @@
     <origin xyz="0 0 ${elbow_length}" rpy="0 0 0"/>
     <axis xyz="0 1 0"/>
-    <limit lower="${-PI/2}" upper="${PI/2}" effort="5.0" velocity="1.0"/>
+    <limit lower="${-PI/2}" upper="${PI/2}" effort="2.0" velocity="0.5"/>
   </joint>
   <!-- Wrist Link (Servo 3) -->
@@ -141,5 +141,5 @@
     <origin xyz="0 0 ${wrist_length}" rpy="0 0 0"/>
     <axis xyz="0 0 1"/>
-    <limit lower="${-PI}" upper="${PI}" effort="5.0" velocity="1.0"/>
+    <limit lower="${-PI}" upper="${PI}" effort="1.5" velocity="0.5"/>
   </joint>
   <!-- Gripper Base Link -->
@@ -169,5 +169,5 @@
     <origin xyz="0 0.015 ${gripper_length/3}" rpy="0 0 0"/>
     <axis xyz="0 1 0"/>
-    <limit lower="0" upper="${PI/4}" effort="2.0" velocity="0.5"/>
+    <limit lower="0" upper="${PI/4}" effort="1.0" velocity="0.3"/>
   </joint>
   <!-- Gripper Left Finger -->
@@ -197,5 +197,5 @@
     <origin xyz="0 -0.015 ${gripper_length/3}" rpy="0 0 0"/>
     <axis xyz="0 1 0"/>
-    <limit lower="${-PI/4}" upper="0" effort="2.0" velocity="0.5"/>
+    <limit lower="${-PI/4}" upper="0" effort="1.0" velocity="0.3"/>
     <mimic joint="gripper_left_joint" multiplier="-1"/>
   </joint>
