Commit message: Fix robot geometry: position wheels at bottom of chassis
- Adjust base_link height to wheel_radius + body_height/2
- Move wheel joints to -body_height/2 (bottom of chassis)
- Update caster positions to match wheel plane
- Fixes issue where wheels appeared in middle of 4-inch chassis

File: source/rpi/ros2-robosort/src/robosort_description/urdf/robosort.urdf.xacro (robot description, xacro)
@@ -79,5 +79,5 @@
     <parent link="base_footprint"/>
     <child link="base_link"/>
-    <origin xyz="0 0 ${wheel_radius}" rpy="0 0 0"/>
+    <origin xyz="0 0 ${wheel_radius + body_height/2}" rpy="0 0 0"/>
   </joint>
   <!-- ============================================ -->
@@ -123,5 +123,5 @@
       <parent link="base_link"/>
       <child link="${prefix}_wheel_link"/>
-      <origin xyz="-0.1 ${reflect*wheel_separation/2} ${-wheel_radius}" rpy="0 0 0"/>
+      <origin xyz="-0.1 ${reflect*wheel_separation/2} ${-body_height/2}" rpy="0 0 0"/>
       <axis xyz="0 1 0"/>
       <limit effort="10.0" velocity="10.0"/>
@@ -163,5 +163,5 @@
       <parent link="base_link"/>
       <child link="${prefix}_caster_link"/>
-      <origin xyz="${reflect_x*caster_offset_x} ${reflect_y*caster_offset_y} ${-wheel_radius + caster_radius}" rpy="0 0 0"/>
+      <origin xyz="${reflect_x*caster_offset_x} ${reflect_y*caster_offset_y} ${-body_height/2 - wheel_radius + caster_radius}" rpy="0 0 0"/>
     </joint>
   </xacro:macro>

Commit message: Update robot colors: wheels black, body gray, LiDAR blue
- Wheels: dark_gray  black
- Body: blue  gray
- LiDAR: black  blue
- Updated both RViz and Gazebo material references

File: source/rpi/ros2-robosort/src/robosort_description/urdf/robosort.urdf.xacro (robot description, xacro)
@@ -36,4 +36,7 @@
     <color rgba="0.3 0.3 0.3 1.0"/>
   </material>
+  <material name="gray">
+    <color rgba="0.5 0.5 0.5 1.0"/>
+  </material>
   <material name="blue">
     <color rgba="0.2 0.4 0.8 1.0"/>
@@ -90,5 +93,5 @@
         <box size="${body_length} ${body_width} ${body_height}"/>
       </geometry>
-      <material name="blue"/>
+      <material name="gray"/>
     </visual>
     <collision>
@@ -110,5 +113,5 @@
           <cylinder radius="${wheel_radius}" length="${wheel_width}"/>
         </geometry>
-        <material name="dark_gray"/>
+        <material name="black"/>
       </visual>
       <collision>
@@ -178,5 +181,5 @@
         <cylinder radius="${lidar_size/2}" length="${lidar_height}"/>
       </geometry>
-      <material name="black"/>
+      <material name="blue"/>
     </visual>
     <collision>
@@ -198,8 +201,8 @@
   <!-- Gazebo colors -->
   <gazebo reference="base_link">
-    <material>Gazebo/Blue</material>
+    <material>Gazebo/Grey</material>
   </gazebo>
   <gazebo reference="left_wheel_link">
-    <material>Gazebo/DarkGrey</material>
+    <material>Gazebo/Black</material>
     <mu1>1.0</mu1>
     <mu2>1.0</mu2>
@@ -210,5 +213,5 @@
   </gazebo>
   <gazebo reference="right_wheel_link">
-    <material>Gazebo/DarkGrey</material>
+    <material>Gazebo/Black</material>
     <mu1>1.0</mu1>
     <mu2>1.0</mu2>
@@ -229,5 +232,5 @@
   </gazebo>
   <gazebo reference="lidar_link">
-    <material>Gazebo/Black</material>
+    <material>Gazebo/Blue</material>
   </gazebo>
   <!-- ============================================ -->

Commit message: Move LiDAR 2 inches forward
- Updated lidar_offset_x from 0.35m to 0.4008m (2 inches forward)
- LiDAR now positioned further ahead on the robot

File: source/rpi/ros2-robosort/src/robosort_description/urdf/robosort.urdf.xacro (robot description, xacro)
@@ -20,5 +20,5 @@
   <xacro:property name="lidar_size" value="0.05"/>
   <xacro:property name="lidar_height" value="0.06"/>
-  <xacro:property name="lidar_offset_x" value="0.35"/>      <!-- Top-front position -->
+  <xacro:property name="lidar_offset_x" value="0.4008"/>     <!-- Top-front position (moved 2 inches forward) -->
   <xacro:property name="lidar_offset_z" value="${body_height/2 + lidar_height/2}"/>
   <!-- Material Properties -->

Commit message: Change LiDAR height to 45mm
- Updated lidar_height from 0.06m to 0.045m (45mm)
- LiDAR now has correct physical dimensions

File: source/rpi/ros2-robosort/src/robosort_description/urdf/robosort.urdf.xacro (robot description, xacro)
@@ -19,5 +19,5 @@
   <!-- LiDAR Properties -->
   <xacro:property name="lidar_size" value="0.05"/>
-  <xacro:property name="lidar_height" value="0.06"/>
+  <xacro:property name="lidar_height" value="0.045"/>     <!-- 45mm height -->
   <xacro:property name="lidar_offset_x" value="0.4008"/>     <!-- Top-front position (moved 2 inches forward) -->
   <xacro:property name="lidar_offset_z" value="${body_height/2 + lidar_height/2}"/>

Commit message: Move wheels backward by 3 inches
- Updated wheel joint X position from -0.1m to -0.1762m
- Wheels now positioned 3 inches further back on the robot

File: source/rpi/ros2-robosort/src/robosort_description/urdf/robosort.urdf.xacro (robot description, xacro)
@@ -126,5 +126,5 @@
       <parent link="base_link"/>
       <child link="${prefix}_wheel_link"/>
-      <origin xyz="-0.1 ${reflect*wheel_separation/2} ${-body_height/2}" rpy="0 0 0"/>
+      <origin xyz="-0.1762 ${reflect*wheel_separation/2} ${-body_height/2}" rpy="0 0 0"/>
       <axis xyz="0 1 0"/>
       <limit effort="10.0" velocity="10.0"/>

Commit message: Update caster wheel dimensions
- Changed caster diameter from 1 inch to 5 inches (radius: 0.025m  0.0635m)
- Set total caster height to 6 inches (extends 6 inches below mounting point)
- Updated caster positioning to accommodate new dimensions

File: source/rpi/ros2-robosort/src/robosort_description/urdf/robosort.urdf.xacro (robot description, xacro)
@@ -14,5 +14,5 @@
   <xacro:property name="wheel_separation" value="0.558"/>   <!-- 22 inches (20 + 2 per side) -->
   <!-- Caster Wheel Properties -->
-  <xacro:property name="caster_radius" value="0.025"/>
+  <xacro:property name="caster_radius" value="0.0635"/>    <!-- 5 inch diameter -->
   <xacro:property name="caster_offset_x" value="0.35"/>     <!-- Front position -->
   <xacro:property name="caster_offset_y" value="0.15"/>     <!-- Left/right spread -->
@@ -166,5 +166,5 @@
       <parent link="base_link"/>
       <child link="${prefix}_caster_link"/>
-      <origin xyz="${reflect_x*caster_offset_x} ${reflect_y*caster_offset_y} ${-body_height/2 - wheel_radius + caster_radius}" rpy="0 0 0"/>
+      <origin xyz="${reflect_x*caster_offset_x} ${reflect_y*caster_offset_y} ${-body_height/2 - 0.1524 + caster_radius}" rpy="0 0 0"/>
     </joint>
   </xacro:macro>

Commit message: Change caster wheels from spheres to cylinders
- Added caster_width property (1 inch width)
- Changed caster geometry from sphere to cylinder
- Updated inertia calculation from sphere to cylinder
- Caster wheels now have realistic cylindrical shape

File: source/rpi/ros2-robosort/src/robosort_description/urdf/robosort.urdf.xacro (robot description, xacro)
@@ -15,4 +15,5 @@
   <!-- Caster Wheel Properties -->
   <xacro:property name="caster_radius" value="0.0635"/>    <!-- 5 inch diameter -->
+  <xacro:property name="caster_width" value="0.025"/>     <!-- 1 inch width -->
   <xacro:property name="caster_offset_x" value="0.35"/>     <!-- Front position -->
   <xacro:property name="caster_offset_y" value="0.15"/>     <!-- Left/right spread -->
@@ -143,5 +144,5 @@
         <origin xyz="0 0 0" rpy="0 0 0"/>
         <geometry>
-          <sphere radius="${caster_radius}"/>
+          <cylinder radius="${caster_radius}" length="${caster_width}"/>
         </geometry>
         <material name="black"/>
@@ -150,5 +151,5 @@
         <origin xyz="0 0 0" rpy="0 0 0"/>
         <geometry>
-          <sphere radius="${caster_radius}"/>
+          <cylinder radius="${caster_radius}" length="${caster_width}"/>
         </geometry>
         <surface>
@@ -161,5 +162,5 @@
         </surface>
       </collision>
-      <xacro:sphere_inertia m="${caster_mass}" r="${caster_radius}"/>
+      <xacro:cylinder_inertia m="${caster_mass}" r="${caster_radius}" h="${caster_width}"/>
     </link>
     <joint name="${prefix}_caster_joint" type="fixed">

Commit message: Rotate caster wheels to match differential drive orientation
- Added 90-degree rotation (PI/2) around X-axis to caster wheels
- Caster wheels now lie flat like drive wheels instead of standing upright
- Position unchanged, only orientation modified

File: source/rpi/ros2-robosort/src/robosort_description/urdf/robosort.urdf.xacro (robot description, xacro)
@@ -142,5 +142,5 @@
     <link name="${prefix}_caster_link">
       <visual>
-        <origin xyz="0 0 0" rpy="0 0 0"/>
+        <origin xyz="0 0 0" rpy="${PI/2} 0 0"/>
         <geometry>
           <cylinder radius="${caster_radius}" length="${caster_width}"/>
@@ -149,5 +149,5 @@
       </visual>
       <collision>
-        <origin xyz="0 0 0" rpy="0 0 0"/>
+        <origin xyz="0 0 0" rpy="${PI/2} 0 0"/>
         <geometry>
           <cylinder radius="${caster_radius}" length="${caster_width}"/>

Commit message: Move differential drive wheels backward by another 3 inches
- Updated wheel X position from -0.1762m to -0.2524m
- Wheels now positioned 6 inches total further back from original position

File: source/rpi/ros2-robosort/src/robosort_description/urdf/robosort.urdf.xacro (robot description, xacro)
@@ -127,5 +127,5 @@
       <parent link="base_link"/>
       <child link="${prefix}_wheel_link"/>
-      <origin xyz="-0.1762 ${reflect*wheel_separation/2} ${-body_height/2}" rpy="0 0 0"/>
+      <origin xyz="-0.2524 ${reflect*wheel_separation/2} ${-body_height/2}" rpy="0 0 0"/>
       <axis xyz="0 1 0"/>
       <limit effort="10.0" velocity="10.0"/>

Commit message: Align caster wheels with rear differential wheels

File: source/rpi/ros2-robosort/src/robosort_description/urdf/robosort.urdf.xacro (robot description, xacro)
@@ -17,5 +17,5 @@
   <xacro:property name="caster_width" value="0.025"/>     <!-- 1 inch width -->
   <xacro:property name="caster_offset_x" value="0.35"/>     <!-- Front position -->
-  <xacro:property name="caster_offset_y" value="0.15"/>     <!-- Left/right spread -->
+  <xacro:property name="caster_offset_y" value="${wheel_separation/2}"/>     <!-- Aligned with drive wheels -->
   <!-- LiDAR Properties -->
   <xacro:property name="lidar_size" value="0.05"/>

Commit message: Fix: Invert LiDAR orientation to correct RViz2 movement direction
- Rotate lidar_link 180 (π) around Z-axis in URDF
- Fixes issue where robot moves forward in real life but backwards in RViz2
- RF2O now calculates correct odometry direction from laser scans

File: source/rpi/ros2-robosort/src/robosort_description/urdf/robosort.urdf.xacro (robot description, xacro)
@@ -195,5 +195,5 @@
     <parent link="base_link"/>
     <child link="lidar_link"/>
-    <origin xyz="${lidar_offset_x} 0 ${lidar_offset_z}" rpy="0 0 0"/>
+    <origin xyz="${lidar_offset_x} 0 ${lidar_offset_z}" rpy="0 0 ${PI}"/>
   </joint>
   <!-- ============================================ -->

Commit message: Revert LiDAR orientation back to original rpy='0 0 0'
- Revert the 180 rotation that was causing movement direction issues
- LiDAR now back to original orientation
- Robot model orientation still needs to be fixed (wheels at front instead of back)

File: source/rpi/ros2-robosort/src/robosort_description/urdf/robosort.urdf.xacro (robot description, xacro)
@@ -195,5 +195,5 @@
     <parent link="base_link"/>
     <child link="lidar_link"/>
-    <origin xyz="${lidar_offset_x} 0 ${lidar_offset_z}" rpy="0 0 ${PI}"/>
+    <origin xyz="${lidar_offset_x} 0 ${lidar_offset_z}" rpy="0 0 0"/>
   </joint>
   <!-- ============================================ -->

Commit message: Move LiDAR to rear position to reverse map orientation

File: source/rpi/ros2-robosort/src/robosort_description/urdf/robosort.urdf.xacro (robot description, xacro)
@@ -21,5 +21,5 @@
   <xacro:property name="lidar_size" value="0.05"/>
   <xacro:property name="lidar_height" value="0.045"/>     <!-- 45mm height -->
-  <xacro:property name="lidar_offset_x" value="0.4008"/>     <!-- Top-front position (moved 2 inches forward) -->
+  <xacro:property name="lidar_offset_x" value="-0.4008"/>     <!-- Top-rear position (moved 2 inches backward) -->
   <xacro:property name="lidar_offset_z" value="${body_height/2 + lidar_height/2}"/>
   <!-- Material Properties -->

Commit message: Move LiDAR to front-left side of robot

File: source/rpi/ros2-robosort/src/robosort_description/urdf/robosort.urdf.xacro (robot description, xacro)
@@ -21,5 +21,6 @@
   <xacro:property name="lidar_size" value="0.05"/>
   <xacro:property name="lidar_height" value="0.045"/>     <!-- 45mm height -->
-  <xacro:property name="lidar_offset_x" value="-0.4008"/>     <!-- Top-rear position (moved 2 inches backward) -->
+  <xacro:property name="lidar_offset_x" value="0.4008"/>     <!-- Top-front position (moved 2 inches forward) -->
+  <xacro:property name="lidar_offset_y" value="0.2"/>       <!-- Left side offset -->
   <xacro:property name="lidar_offset_z" value="${body_height/2 + lidar_height/2}"/>
   <!-- Material Properties -->
@@ -195,5 +196,5 @@
     <parent link="base_link"/>
     <child link="lidar_link"/>
-    <origin xyz="${lidar_offset_x} 0 ${lidar_offset_z}" rpy="0 0 0"/>
+    <origin xyz="${lidar_offset_x} ${lidar_offset_y} ${lidar_offset_z}" rpy="0 0 0"/>
   </joint>
   <!-- ============================================ -->

Commit message: Center LiDAR in front of robot

File: source/rpi/ros2-robosort/src/robosort_description/urdf/robosort.urdf.xacro (robot description, xacro)
@@ -22,5 +22,4 @@
   <xacro:property name="lidar_height" value="0.045"/>     <!-- 45mm height -->
   <xacro:property name="lidar_offset_x" value="0.4008"/>     <!-- Top-front position (moved 2 inches forward) -->
-  <xacro:property name="lidar_offset_y" value="0.2"/>       <!-- Left side offset -->
   <xacro:property name="lidar_offset_z" value="${body_height/2 + lidar_height/2}"/>
   <!-- Material Properties -->
@@ -196,5 +195,5 @@
     <parent link="base_link"/>
     <child link="lidar_link"/>
-    <origin xyz="${lidar_offset_x} ${lidar_offset_y} ${lidar_offset_z}" rpy="0 0 0"/>
+    <origin xyz="${lidar_offset_x} 0 ${lidar_offset_z}" rpy="0 0 0"/>
   </joint>
   <!-- ============================================ -->

Commit message: Fix wheel joint axes for correct forward/backward motion

File: source/rpi/ros2-robosort/src/robosort_description/urdf/robosort.urdf.xacro (robot description, xacro)
@@ -128,5 +128,5 @@
       <child link="${prefix}_wheel_link"/>
       <origin xyz="-0.2524 ${reflect*wheel_separation/2} ${-body_height/2}" rpy="0 0 0"/>
-      <axis xyz="0 1 0"/>
+      <axis xyz="0 ${reflect} 0"/>
       <limit effort="3.0" velocity="1.4"/>
       <dynamics damping="0.5" friction="0.3"/>

Commit message: Fix wheel macro to use explicit axis parameters

File: source/rpi/ros2-robosort/src/robosort_description/urdf/robosort.urdf.xacro (robot description, xacro)
@@ -107,5 +107,5 @@
   <!-- Wheel Macro -->
   <!-- ============================================ -->
-  <xacro:macro name="wheel" params="prefix reflect">
+  <xacro:macro name="wheel" params="prefix reflect axis">
     <link name="${prefix}_wheel_link">
       <visual>
@@ -128,5 +128,5 @@
       <child link="${prefix}_wheel_link"/>
       <origin xyz="-0.2524 ${reflect*wheel_separation/2} ${-body_height/2}" rpy="0 0 0"/>
-      <axis xyz="0 ${reflect} 0"/>
+      <axis xyz="${axis}"/>
       <limit effort="3.0" velocity="1.4"/>
       <dynamics damping="0.5" friction="0.3"/>
@@ -134,6 +134,6 @@
   </xacro:macro>
   <!-- Left and Right Drive Wheels -->
-  <xacro:wheel prefix="left" reflect="1"/>
-  <xacro:wheel prefix="right" reflect="-1"/>
+  <xacro:wheel prefix="left" reflect="1" axis="0 1 0"/>
+  <xacro:wheel prefix="right" reflect="-1" axis="0 -1 0"/>
   <!-- ============================================ -->
   <!-- Caster Wheel Macro -->

Commit message: Revert wheel axes to original for correct motion

File: source/rpi/ros2-robosort/src/robosort_description/urdf/robosort.urdf.xacro (robot description, xacro)
@@ -107,5 +107,5 @@
   <!-- Wheel Macro -->
   <!-- ============================================ -->
-  <xacro:macro name="wheel" params="prefix reflect axis">
+  <xacro:macro name="wheel" params="prefix reflect">
     <link name="${prefix}_wheel_link">
       <visual>
@@ -128,5 +128,5 @@
       <child link="${prefix}_wheel_link"/>
       <origin xyz="-0.2524 ${reflect*wheel_separation/2} ${-body_height/2}" rpy="0 0 0"/>
-      <axis xyz="${axis}"/>
+      <axis xyz="0 1 0"/>
       <limit effort="3.0" velocity="1.4"/>
       <dynamics damping="0.5" friction="0.3"/>
@@ -134,6 +134,6 @@
   </xacro:macro>
   <!-- Left and Right Drive Wheels -->
-  <xacro:wheel prefix="left" reflect="1" axis="0 1 0"/>
-  <xacro:wheel prefix="right" reflect="-1" axis="0 -1 0"/>
+  <xacro:wheel prefix="left" reflect="1"/>
+  <xacro:wheel prefix="right" reflect="-1"/>
   <!-- ============================================ -->
   <!-- Caster Wheel Macro -->
